Commit message: "created core urdf file for RAKSH"

File: description/robot_core.xacro (robot description, xacro)
@@ -1,4 +1,5 @@
 <?xml version="1.0"?>
 <robot xmlns:xacro="http://www.ros.org/wiki/xacro"  name="robot">
+    <xacro:include filename="inertia_macros.xacro"/>
     <material name="white">
         <color rgba="1 1 1 1"/>
@@ -26,17 +27,26 @@
             <origin xyz="0.3 0 0.1"/>
             <geometry>
-                <box size="0.6 0.4 0.2"/>
+                <box size="0.8 0.4 0.2"/>
             </geometry>
             <material name="white"/>
         </visual>
+        <collision>
+                <origin xyz="0.3 0 0.1"/>
+                <geometry>
+                    <box size="0.8 0.4 0.2"/>
+                </geometry>
+        </collision>
+        <xacro:inertial_box mass="1.25" x='0.8' y="0.4" z="0.2">
+            <origin xyz="0.3 0 0.1" rpy="0.0 0.0 0.0"/>
+        </xacro:inertial_box>
     </link>
-    <!-- Left Wheel Link -->
-    <joint name="left_wheel_joint" type="continuous">
+    <!-- Left Wheel Link1 -->
+    <joint name="left_wheel_joint1" type="continuous">
         <parent link="base_link"/>
-        <child link="left_wheel"/>
+        <child link="left_wheel1"/>
         <origin xyz="0 0.225 0" rpy="-${pi/2} 0.0 0.0"/>
         <axis xyz="0 0 1"/>
     </joint>
-    <link name="left_wheel">
+    <link name="left_wheel1">
         <visual>
             <geometry>
@@ -45,19 +55,123 @@
             <material name="blue"></material>
         </visual>
+        <collision>
+            <geometry>
+                <cylinder radius="0.08" length="0.04"/>
+            </geometry>
+        </collision>
+        <xacro:inertial_cylinder mass="0.1" length="0.04" radius="0.08">
+            <origin xyz="0.0 0.0 0.0" rpy="0.0 0.0 0.0"/>
+        </xacro:inertial_cylinder>
+    </link>
+    <joint name="left_wheel_joint2" type="continuous">
+        <parent link="base_link"/>
+        <child link="left_wheel2"/>
+        <origin xyz="0.2 0.225 0" rpy="-${pi/2} 0.0 0.0"/>
+        <axis xyz="0 0 1"/>
+    </joint>
+    <link name="left_wheel2">
+        <visual>
+            <geometry>
+                <cylinder radius="0.08" length="0.04"/>
+            </geometry>
+            <material name="blue"></material>
+        </visual>
+        <collision>
+            <geometry>
+                <cylinder radius="0.08" length="0.04"/>
+            </geometry>
+        </collision>
+        <xacro:inertial_cylinder mass="0.1" length="0.04" radius="0.08">
+            <origin xyz="0.0 0.0 0.0" rpy="0.0 0.0 0.0"/>
+        </xacro:inertial_cylinder>
+    </link>
+    <joint name="left_wheel_joint3" type="continuous">
+        <parent link="base_link"/>
+        <child link="left_wheel3"/>
+        <origin xyz="0.5 0.225 0" rpy="-${pi/2} 0.0 0.0"/>
+        <axis xyz="0 0 1"/>
+    </joint>
+    <link name="left_wheel3">
+        <visual>
+            <geometry>
+                <cylinder radius="0.08" length="0.04"/>
+            </geometry>
+            <material name="blue"></material>
+        </visual>
+        <collision>
+            <geometry>
+                <cylinder radius="0.08" length="0.04"/>
+            </geometry>
+        </collision>
+        <xacro:inertial_cylinder mass="0.1" length="0.04" radius="0.08">
+            <origin xyz="0.0 0.0 0.0" rpy="0.0 0.0 0.0"/>
+        </xacro:inertial_cylinder>
     </link>
         <!-- right Wheel Link -->
-        <joint name="right_wheel_joint" type="continuous">
-            <parent link="base_link"/>
-            <child link="right_wheel"/>
-            <origin xyz="0 -0.225 0" rpy="+${pi/2} 0.0 0.0"/>
-            <axis xyz="0 0 -1"/>
-        </joint>
-        <link name="right_wheel">
-            <visual>
-                <geometry>
-                    <cylinder radius="0.08" length="0.04"/>
-                </geometry>
-                <material name="blue"></material>
-            </visual>
-        </link>
+    <joint name="right_wheel_joint1" type="continuous">
+        <parent link="base_link"/>
+        <child link="right_wheel1"/>
+        <origin xyz="0 -0.225 0" rpy="+${pi/2} 0.0 0.0"/>
+        <axis xyz="0 0 -1"/>
+    </joint>
+    <link name="right_wheel1">
+        <visual>
+            <geometry>
+                <cylinder radius="0.08" length="0.04"/>
+            </geometry>
+            <material name="blue"></material>
+        </visual>
+        <collision>
+            <geometry>
+                <cylinder radius="0.08" length="0.04"/>
+            </geometry>
+        </collision>
+        <xacro:inertial_cylinder mass="0.1" length="0.04" radius="0.08">
+            <origin xyz="0.0 0.0 0.0" rpy="0.0 0.0 0.0"/>
+        </xacro:inertial_cylinder>
+    </link>
+    <joint name="right_wheel_joint2" type="continuous">
+        <parent link="base_link"/>
+        <child link="right_wheel2"/>
+        <origin xyz="0.2 -0.225 0" rpy="+${pi/2} 0.0 0.0"/>
+        <axis xyz="0 0 -1"/>
+    </joint>
+    <link name="right_wheel2">
+        <visual>
+            <geometry>
+                <cylinder radius="0.08" length="0.04"/>
+            </geometry>
+            <material name="blue"></material>
+        </visual>
+        <collision>
+            <geometry>
+                <cylinder radius="0.08" length="0.04"/>
+            </geometry>
+        </collision>
+        <xacro:inertial_cylinder mass="0.1" length="0.04" radius="0.08">
+            <origin xyz="0.0 0.0 0.0" rpy="0.0 0.0 0.0"/>
+        </xacro:inertial_cylinder>
+    </link>
+    <joint name="right_wheel_joint3" type="continuous">
+        <parent link="base_link"/>
+        <child link="right_wheel3"/>
+        <origin xyz="0.5 -0.225 0" rpy="+${pi/2} 0.0 0.0"/>
+        <axis xyz="0 0 -1"/>
+    </joint>
+    <link name="right_wheel3">
+        <visual>
+            <geometry>
+                <cylinder radius="0.08" length="0.04"/>
+            </geometry>
+            <material name="blue"></material>
+        </visual>
+        <collision>
+            <geometry>
+                <cylinder radius="0.08" length="0.04"/>
+            </geometry>
+        </collision>
+        <xacro:inertial_cylinder mass="0.1" length="0.04" radius="0.08">
+            <origin xyz="0.0 0.0 0.0" rpy="0.0 0.0 0.0"/>
+        </xacro:inertial_cylinder>
+    </link>
 </robot>

Commit message: "Added Gazebo simulation and controls"

File: description/robot_core.xacro (robot description, xacro)
@@ -41,4 +41,9 @@
         </xacro:inertial_box>
     </link>
+    <gazebo reference="chassis">
+        <material>
+            Gazebo/White
+        </material>
+    </gazebo>
     <!-- Left Wheel Link1 -->
     <joint name="left_wheel_joint1" type="continuous">
@@ -64,4 +69,9 @@
         </xacro:inertial_cylinder>
     </link>
+    <gazebo reference="left_wheel1">
+        <material>
+            Gazebo/Blue
+        </material>
+    </gazebo>
     <joint name="left_wheel_joint2" type="continuous">
         <parent link="base_link"/>
@@ -86,4 +96,9 @@
         </xacro:inertial_cylinder>
     </link>
+    <gazebo reference="left_wheel2">
+        <material>
+            Gazebo/Blue
+        </material>
+    </gazebo>
     <joint name="left_wheel_joint3" type="continuous">
         <parent link="base_link"/>
@@ -108,4 +123,9 @@
         </xacro:inertial_cylinder>
     </link>
+    <gazebo reference="left_wheel3">
+        <material>
+            Gazebo/Blue
+        </material>
+    </gazebo>
         <!-- right Wheel Link -->
     <joint name="right_wheel_joint1" type="continuous">
@@ -131,4 +151,9 @@
         </xacro:inertial_cylinder>
     </link>
+    <gazebo reference="right_wheel1">
+        <material>
+            Gazebo/Blue
+        </material>
+    </gazebo>
     <joint name="right_wheel_joint2" type="continuous">
         <parent link="base_link"/>
@@ -153,4 +178,9 @@
         </xacro:inertial_cylinder>
     </link>
+    <gazebo reference="right_wheel2">
+        <material>
+            Gazebo/Blue
+        </material>
+    </gazebo>
     <joint name="right_wheel_joint3" type="continuous">
         <parent link="base_link"/>
@@ -175,3 +205,8 @@
         </xacro:inertial_cylinder>
     </link>
+    <gazebo reference="right_wheel3">
+        <material>
+            Gazebo/Blue
+        </material>
+    </gazebo>
 </robot>

Commit message: "Set up the Lidar for robot"

File: description/robot_core.xacro (robot description, xacro)
@@ -14,4 +14,7 @@
         <color rgba="0 0 0 1"/>
     </material>
+    <material name="red">
+        <color rgba="1 0 0 01"/>
+    </material>
     <!-- Base link -->
     <link name="base_link">
