Commit message: done till EKF

File: ugv_ws/src/ugv_description/urdf/ugv.urdf.xacro (robot description, xacro)
@@ -165,26 +165,39 @@
     </sensor>
   </gazebo>
-  <!-- Camera Sensor -->
-  <link name="camera_left_link">
-    <inertial>
-      <mass value="0.001"/>
-      <inertia ixx="0.000001" ixy="0" ixz="0" iyy="0.000001" iyz="0" izz="0.000001"/>
-    </inertial>
-  </link>
-  <joint name="camera_left_joint" type="fixed">
-    <parent link="camera_link"/>
-    <child  link="camera_left_link"/>
-    <origin xyz="0 0.06 0" rpy="${-PI/2} 0 ${-PI/2}"/>
-  </joint>
-  <link name="camera_right_link">
-    <inertial>
-      <mass value="0.001"/>
-      <inertia ixx="0.000001" ixy="0" ixz="0" iyy="0.000001" iyz="0" izz="0.000001"/>
-    </inertial>
-  </link>
-  <joint name="camera_right_joint" type="fixed">
-    <parent link="camera_link"/>
-    <child  link="camera_right_link"/>
-    <origin xyz="0 -0.06 0" rpy="${-PI/2} 0 ${-PI/2}"/>
-  </joint>
+  <!-- Left camera -->
+  <gazebo reference="camera_left_link">
+    <sensor name="camera_left" type="camera">
+      <always_on>true</always_on>
+      <update_rate>30</update_rate>
+      <topic>camera/left/image_raw</topic>
+      <gz_frame_id>camera_left_link</gz_frame_id>
+      <camera>
+        <horizontal_fov>1.3962634</horizontal_fov>
+        <image>
+          <width>640</width>
+          <height>480</height>
+          <format>RGB_INT8</format>
+        </image>
+        <clip><near>0.02</near><far>30.0</far></clip>
+      </camera>
+    </sensor>
+  </gazebo>
+  <!-- Right camera -->
+  <gazebo reference="camera_right_link">
+    <sensor name="camera_right" type="camera">
+      <always_on>true</always_on>
+      <update_rate>30</update_rate>
+      <topic>camera/right/image_raw</topic>
+      <gz_frame_id>camera_right_link</gz_frame_id>
+      <camera>
+        <horizontal_fov>1.3962634</horizontal_fov>
+        <image>
+          <width>640</width>
+          <height>480</height>
+          <format>RGB_INT8</format>
+        </image>
+        <clip><near>0.02</near><far>30.0</far></clip>
+      </camera>
+    </sensor>
+  </gazebo>
 </robot>

Commit message: trying to fix slam

File: ugv_ws/src/ugv_description/urdf/ugv.urdf.xacro (robot description, xacro)
@@ -92,4 +92,22 @@
     <origin xyz="0.0 0.0 0.05" rpy="0 0 0"/>
   </joint>
+  <!-- ===== LIDAR (for Nav2 costmap) ===== -->
+  <link name="lidar_link">
+    <visual>
+      <geometry><cylinder length="0.02" radius="0.03"/></geometry>
+      <material name="black"><color rgba="0.1 0.1 0.1 1"/></material>
+    </visual>
+    <inertial>
+      <mass value="0.05"/>
+      <inertia ixx="0.000001" ixy="0" ixz="0"
+               iyy="0.000001" iyz="0"
+               izz="0.000001"/>
+    </inertial>
+  </link>
+  <joint name="lidar_joint" type="fixed">
+    <parent link="base_link"/>
+    <child  link="lidar_link"/>
+    <origin xyz="0.0 0.0 0.08" rpy="0 0 0"/>
+  </joint>
   <!-- ===== STEREO CAMERA MOUNT ===== -->
   <link name="camera_link">
@@ -165,4 +183,28 @@
     </sensor>
   </gazebo>
+  <!-- Lidar sensor for Nav2 costmap -->
+  <gazebo reference="lidar_link">
+    <sensor name="lidar" type="gpu_lidar">
+      <always_on>true</always_on>
+      <update_rate>10</update_rate>
+      <topic>scan</topic>
+      <gz_frame_id>lidar_link</gz_frame_id>
+      <lidar>
+        <scan>
+          <horizontal>
+            <samples>360</samples>
+            <resolution>1</resolution>
+            <min_angle>-3.14159</min_angle>
+            <max_angle>3.14159</max_angle>
+          </horizontal>
+        </scan>
+        <range>
+          <min>0.1</min>
+          <max>10.0</max>
+          <resolution>0.01</resolution>
+        </range>
+      </lidar>
+    </sensor>
+  </gazebo>
   <!-- Left camera -->
   <gazebo reference="camera_left_link">
@@ -180,4 +222,13 @@
         </image>
         <clip><near>0.02</near><far>30.0</far></clip>
+        <lens>
+          <intrinsics>
+            <fx>381.361</fx>
+            <fy>381.361</fy>
+            <cx>320.0</cx>
+            <cy>240.0</cy>
+            <s>0</s>
+          </intrinsics>
+        </lens>
       </camera>
     </sensor>
@@ -198,4 +249,13 @@
         </image>
         <clip><near>0.02</near><far>30.0</far></clip>
+        <lens>
+          <intrinsics>
+            <fx>381.361</fx>
+            <fy>381.361</fy>
+            <cx>320.0</cx>
+            <cy>240.0</cy>
+            <s>0</s>
+          </intrinsics>
+        </lens>
       </camera>
     </sensor>
